Commit message: Resetting robot model

File: robot_description/urdf/common_properties.urdf.xacro (robot description, xacro)
@@ -25,3 +25,57 @@
 	<xacro:property name="cam_op" value="0" />
 	<xacro:property name="cam_oy" value="0" />
+<!--
+  Various useful properties such as constants and materials
+-->
+  <xacro:property name="M_PI" value="3.1415926535897931" />
+  <xacro:property name="material_white">
+    <material name="white">
+      <color rgba="1 1 1 1"/>
+    </material>
+  </xacro:property>
+  <xacro:property name="material_grey">
+    <material name="grey">
+      <color rgba="0.5 0.5 0.5 1"/>
+    </material>
+  </xacro:property>
+  <xacro:property name="material_light_grey">
+    <material name="light_grey">
+      <color rgba="0.6 0.6 0.6 1"/>
+    </material>
+  </xacro:property>
+  <xacro:property name="material_dark_grey">
+    <material name="dark_grey">
+      <color rgba="0.3 0.3 0.3 1"/>
+    </material>
+  </xacro:property>
+  <xacro:property name="material_black">
+    <material name="black">
+      <color rgba="0.1 0.1 0.1 1"/>
+    </material>
+  </xacro:property>
+  <xacro:property name="material_red">
+    <material name="red">
+      <color rgba="1 0 0 1"/>
+    </material>
+  </xacro:property>
+  <xacro:property name="material_green">
+    <material name="green">
+      <color rgba="0.0 0.8 0.0 1"/>
+    </material>
+  </xacro:property>
+  <xacro:property name="material_blue">
+    <material name="blue">
+      <color rgba="0.0 0.0 1.0 1"/>
+    </material>
+  </xacro:property>
+  <xacro:property name="material_grey_blue">
+    <material name="grey_blue">
+      <color rgba="0.4 0.4 1.0 1"/>
+    </material>
+  </xacro:property>
+  <xacro:property name="material_orange">
+    <material name="orange">
+      <color rgba="1.0 0.7 0.0 1"/>
+    </material>
+  </xacro:property>
 </robot>

File: robot_description/urdf/sensors/r200.urdf.xacro (robot description, xacro)
@@ -1,7 +1,17 @@
 <?xml version="1.0"?>
 <robot name="sensor_r200" xmlns:xacro="http://ros.org/wiki/xacro">
-  <xacro:include filename="$(find turtlebot_description)/urdf/turtlebot_gazebo.urdf.xacro"/>
-  <xacro:include filename="$(find turtlebot_description)/urdf/turtlebot_properties.urdf.xacro"/>
-  <!-- Camera parameters -->
+  <xacro:include filename="$(find robot_description)/urdf/turtlebot_gazebo.urdf.xacro"/>
+  <xacro:include filename="$(find robot_description)/urdf/turtlebot_properties.urdf.xacro"/>
+  <!-- Mount and camera parameters -->
+  <xacro:property name="pole_px" value="-0.103" />
+  <xacro:property name="pole_py" value="-0.098"/>
+  <xacro:property name="pole_pz" value="0.269" />
+  <xacro:property name="r200_bracket_end_offset_py" value="0.02" />
+  <xacro:property name="r200_bracket_end_offset_pz" value="0" />
+  <xacro:property name="r200_bracket_end_width"     value="0.026" />
+  <xacro:property name="r200_bracket_offset_py" value="0.010" />
+  <xacro:property name="r200_bracket_offset_pz" value="0.010" />
+  <xacro:property name="r200_bracket_length"    value="0.176" />
+  <xacro:property name="r200_bracket_width"     value="0.0285" />
   <xacro:property name="r200_cam_offset_px" value="-0.017" />
   <xacro:property name="r200_cam_offset_py" value="0.024" />
@@ -13,12 +23,62 @@
   <xacro:macro name="sensor_r200" params="parent">
     <!--
-    ==  Camera body joints & links ==
+    ==  Mount and camera body joints & links ==
     -->
+    <!-- right bracket end -->
+    <joint name="bracket_end_right_joint" type="fixed">
+      <origin xyz="${pole_px} ${pole_py} ${pole_pz}" rpy="0 0 0"/>
+      <parent link="${parent}"/>
+      <child link="bracket_end_right" />
+    </joint>
+    <link name="bracket_end_right">
+    <visual>
+       <origin xyz="${-r200_bracket_end_width/2} ${r200_bracket_end_offset_py} ${r200_bracket_end_offset_pz}" rpy="0 0 ${-M_PI/2}"/>
+        <geometry>
+         <mesh filename="package://robot_description/meshes/sensors/r200_bracket_end.stl" scale="0.001 0.001 0.001"/>
+        </geometry>
+        <xacro:insert_block name="material_dark_grey" />
+      </visual>
+    </link>
+    <!-- center main bracket -->
+    <joint name="bracket_joint" type="fixed">
+      <origin xyz="${r200_bracket_width/2} ${r200_bracket_offset_py} ${r200_bracket_offset_pz}" rpy="0 0 0"/>
+      <parent link="bracket_end_right"/>
+      <child link="bracket" />
+    </joint>
+    <link name="bracket">
+    <visual>
+       <origin xyz="0 0 0" rpy="0 0 ${M_PI/2}"/>
+        <geometry>
+         <mesh filename="package://robot_description/meshes/sensors/r200_bracket.stl" scale="0.001 0.001 0.001"/>
+        </geometry>
+        <xacro:insert_block name="material_dark_grey" />
+      </visual>
+    </link>
+    <!-- left bracket end -->
+    <joint name="bracket_end_left_joint" type="fixed">
+      <origin xyz="${-r200_bracket_width/2} ${r200_bracket_length - r200_bracket_offset_py} ${-r200_bracket_offset_pz}" rpy="0 0 0"/>
+      <parent link="bracket"/>
+      <child link="bracket_end_left" />
+    </joint>
+    <link name="bracket_end_left">
+    <visual>
+       <origin xyz="${r200_bracket_end_width/2} 0 ${-r200_bracket_end_offset_pz}" rpy="0 0 ${M_PI/2}"/>
+        <geometry>
+         <mesh filename="package://robot_description/meshes/sensors/r200_bracket_end.stl" scale="0.001 0.001 0.001"/>
+        </geometry>
+        <xacro:insert_block name="material_dark_grey" />
+      </visual>
+    </link>
     <!-- camera body -->
+    <joint name="camera_joint" type="fixed">
+      <origin xyz="${r200_cam_offset_px} ${r200_cam_offset_py} ${r200_cam_offset_pz}" rpy="0 0 0"/>
+      <parent link="bracket"/>
+      <child link="camera_link" />
+    </joint>
     <link name="camera_link">
       <visual>
        <origin xyz="0 0 0" rpy="${M_PI/2} 0 ${M_PI/2}"/>
         <geometry>
-         <mesh filename="package://turtlebot_description/meshes/sensors/r200.dae" />
+         <mesh filename="package://robot_description/meshes/sensors/r200.dae" />
         </geometry>
       </visual>

File: robot_description/urdf/stacks/hexagons.urdf.xacro (robot description, xacro)
@@ -4,5 +4,5 @@
  -->
 <robot name="stack_hexagons" xmlns:xacro="http://ros.org/wiki/xacro">
-  <xacro:include filename="$(find turtlebot_description)/urdf/common_properties.urdf.xacro"/>
+  <xacro:include filename="$(find robot_description)/urdf/common_properties.urdf.xacro"/>
   <!-- Xacro properties -->
   <xacro:property name="M_SCALE" value="0.001"/>
@@ -19,5 +19,5 @@
         <origin xyz="0 0 0" rpy="0 0 0"/>
         <geometry>
-          <mesh filename="package://turtlebot_description/meshes/stacks/hexagons/pole_bottom.dae"/>
+          <mesh filename="package://robot_description/meshes/stacks/hexagons/pole_bottom.dae"/>
         </geometry>
       </visual>
@@ -47,5 +47,5 @@
         <origin xyz="0 0 0" rpy="0 ${M_PI} 0"/>
         <geometry>
-          <mesh filename="package://turtlebot_description/meshes/stacks/hexagons/pole_middle.dae"/>
+          <mesh filename="package://robot_description/meshes/stacks/hexagons/pole_middle.dae"/>
         </geometry>
       </visual>
@@ -75,5 +75,5 @@
         <origin xyz=" 0 0 0" rpy="0 0 0"/>
         <geometry>
-          <mesh filename="package://turtlebot_description/meshes/stacks/hexagons/pole_top.dae"/>
+          <mesh filename="package://robot_description/meshes/stacks/hexagons/pole_top.dae"/>
         </geometry>
       </visual>
@@ -103,5 +103,5 @@
         <origin xyz="0 0 -0.01" rpy="0 0 0"/>
         <geometry>
-          <mesh filename="package://turtlebot_description/meshes/sensors/sensor_pole.dae" />
+          <mesh filename="package://robot_description/meshes/sensors/sensor_pole.dae" />
         </geometry>
       </visual>
@@ -142,5 +142,5 @@
         <origin xyz="0 0 0" rpy="0 0 0"/>
         <geometry>
-          <mesh filename="package://turtlebot_description/meshes/stacks/hexagons/plate_bottom.dae"/>
+          <mesh filename="package://robot_description/meshes/stacks/hexagons/plate_bottom.dae"/>
         </geometry>
       </visual>
@@ -172,5 +172,5 @@
         <origin xyz="0 0 0" rpy="0 0 0"/>
         <geometry>
-          <mesh filename="package://turtlebot_description/meshes/stacks/hexagons/plate_middle.dae"/>
+          <mesh filename="package://robot_description/meshes/stacks/hexagons/plate_middle.dae"/>
         </geometry>
       </visual>
@@ -204,5 +204,5 @@
         <origin xyz="0 0 0" rpy="0 0 0"/>
         <geometry>
-          <mesh filename="package://turtlebot_description/meshes/stacks/hexagons/plate_top.dae"/>
+          <mesh filename="package://robot_description/meshes/stacks/hexagons/plate_top.dae"/>
         </geometry>
       </visual>

Commit message: Updating robot model

File: robot_description/urdf/common_properties.urdf.xacro (robot description, xacro)
@@ -79,3 +79,8 @@
     </material>
   </xacro:property>
+  <xacro:property name="material_aluminum">
+    <material name="aluminum">
+	    <color rgba="0.5 0.5 0.5 1"/>
+    </material>
+  </xacro:property>
 </robot>

File: robot_description/urdf/kobuki.urdf.xacro (robot description, xacro)
@@ -8,5 +8,5 @@
 <robot name="kobuki" xmlns:xacro="http://ros.org/wiki/xacro">
   <xacro:include filename="$(find robot_description)/urdf/common_properties.urdf.xacro"/>
-  <xacro:include filename="$(find robot_description)/urdf/kobuki_gazebo.urdf.xacro"/>
+  <!-- <xacro:include filename="$(find robot_description)/urdf/kobuki_gazebo.urdf.xacro"/> -->
   <!-- Kobuki -->
   <xacro:macro name="kobuki">
@@ -209,5 +209,5 @@
     </link>
     <!-- Kobuki Gazebo simulation details -->
-    <kobuki_sim/>
+    <!-- <kobuki_sim/> -->
   </xacro:macro>
 </robot>

File: robot_description/urdf/sensors/rplidar.urdf.xacro (robot description, xacro)
@@ -1,5 +1,4 @@
 <?xml version="1.0"?>
 <robot xmlns:xacro="http://www.ros.org/wiki/xacro">
-    <xacro:property name="M_PI" value="3.1415926535897931" />
     <xacro:macro name="rplidar_model" params="name parent *origin">
       <joint name="${name}_joint" type="fixed">
@@ -12,10 +11,12 @@
           <mass value="0.270" />
           <origin xyz="0 0 0" rpy="0 0 0" />
-          <inertia ixx="2.632e-4" ixy="0" ixz="0" iyy="2.632e-4" iyz="0" izz="1.62e-4" />
+          <inertia ixx="2.632e-4" ixy="0" ixz="0"
+                   iyy="2.632e-4" iyz="0"
+                   izz="1.62e-4" />
         </inertial>
         <visual>
           <origin xyz="0 0 0" rpy="0 0 0" />
           <geometry>
-          <mesh filename="package://hector_sensors_description/meshes/hokuyo_utm30lx/hokuyo_utm_30lx.dae"/>
+          <mesh filename="package://robot_description/meshes/rplidar_a2.stl"/>
         </geometry>
         </visual>
@@ -32,36 +33,4 @@
         <xacro:insert_block name="origin" />
       </xacro:rplidar_model>
-      <gazebo reference="${name}_frame">
-        <sensor type="ray" name="${name}">
-          <always_on>true</always_on>
-          <update_rate>${update_rate}</update_rate>
-          <pose>0 0 0 0 0 0</pose>
-          <visualize>false</visualize>
-          <ray>
-            <scan>
-              <horizontal>
-                <samples>${ray_count}</samples>
-                <resolution>1</resolution>
-                <min_angle>${min_angle * M_PI/180}</min_angle>
-                <max_angle>${max_angle * M_PI/180}</max_angle>
-              </horizontal>
-            </scan>
-            <range>
-              <min>0.2</min>
-              <max>15.0</max>
-              <resolution>0.01</resolution>
-            </range>
-            <noise>
-              <type>gaussian</type>
-              <mean>0.0</mean>
-              <stddev>0.004</stddev>
-            </noise>
-          </ray>
-          <plugin name="gazebo_ros_${name}_controller" filename="libgazebo_ros_laser.so">
-            <topicName>${ros_topic}</topicName>
-            <frameName>${name}_frame</frameName>
-          </plugin>
-        </sensor>
-      </gazebo>
     </xacro:macro>
 </robot>
