Commit message: final updates to model

File: robot_description/robots/kobuki_hexagons_d435.xacro (robot description, xacro)
@@ -6,13 +6,17 @@
 -->
 <robot name="robot" xmlns:xacro="http://ros.org/wiki/xacro">
-  <!-- <xacro:include filename="$(find robot_description)/urdf/turtlebot_common_library.urdf.xacro" /> -->
-  <!-- <xacro:include filename="$(find robot_description)/urdf/kobuki.urdf.xacro" /> -->
-  <!-- <xacro:include filename="$(find robot_description)/urdf/stacks/hexagons.urdf.xacro"/> -->
+  <xacro:include filename="$(find robot_description)/urdf/kobuki.urdf.xacro" />
+  <xacro:include filename="$(find robot_description)/urdf/stacks/custom_hexagons.urdf.xacro"/>
   <xacro:include filename="$(find robot_description)/urdf/sensors/d435.urdf.xacro"/>
-  <!-- <kobuki/> -->
-  <!-- <stack_hexagons parent="base_link"/> -->
-  <link name="base_link" />
-  <sensor_d435 parent="base_link">
-    <origin xyz="0 0 0" rpy="0 0 0"/>
+  <xacro:include filename="$(find robot_description)/urdf/sensors/rplidar.urdf.xacro"/>
+  <kobuki/>
+  <!-- FOR TESTING -->
+  <!-- <link name="base_link" /> -->
+  <stack_hexagons parent="base_link"/>
+  <sensor_d435 parent="plate_bottom_link">
+    <origin xyz="0.115 0 0.0025" rpy="0 0 0"/>
   </sensor_d435>
+  <rplidar parent="plate_middle_link">
+    <origin xyz="0 0 0.0025" rpy="0 0 0"/>
+  </rplidar>
 </robot>

File: robot_description/urdf/common_properties.urdf.xacro (robot description, xacro)
@@ -8,24 +8,6 @@
    -->
   <!--
-   ======================================================================
-   - REP 119 : Rgb camera link relative to the Base link
-   ======================================================================
-     Base link is currently defined as the rotational centre on the bottom
-     of the base mould. For both create and kobuki this is actually exactly
-     the same 3d world point.
-     This may cause an issue with a base with much different floor clearance.
-     Should we be using base_footprint for this specification instead?
-     Note: REP needs to be updated with the information below
-     (currently in development and awaiting feedback)
-   -->
-	<xacro:property name="cam_px" value="-0.087" />
-<!--	<xacro:property name="cam_py" value="-0.0125" /> Y varies for different configurations. get sets in sensors_urdf -->
-	<xacro:property name="cam_pz" value="0.2870" />
-	<xacro:property name="cam_or" value="0" />
-	<xacro:property name="cam_op" value="0" />
-	<xacro:property name="cam_oy" value="0" />
-<!--
-  Various useful properties such as constants and materials
--->
+    Various useful properties such as constants and materials
+  -->
   <xacro:property name="M_PI" value="3.1415926535897931" />
   <xacro:property name="material_white">

File: robot_description/urdf/kobuki.urdf.xacro (robot description, xacro)
@@ -8,5 +8,4 @@
 <robot name="kobuki" xmlns:xacro="http://ros.org/wiki/xacro">
   <xacro:include filename="$(find robot_description)/urdf/common_properties.urdf.xacro"/>
-  <!-- <xacro:include filename="$(find robot_description)/urdf/kobuki_gazebo.urdf.xacro"/> -->
   <!-- Kobuki -->
   <xacro:macro name="kobuki">
@@ -43,5 +42,5 @@
         <!-- COM experimentally determined -->
         <origin xyz="0.01 0 0"/>
-        <mass value="2.4"/> <!-- 2.4/2.6 kg for small/big battery pack -->
+        <mass value="2.6"/> <!-- 2.4/2.6 kg for small/big battery pack -->
         <!-- Kobuki's inertia tensor is approximated by a cylinder with homogeneous mass distribution
              More details: http://en.wikipedia.org/wiki/List_of_moment_of_inertia_tensors
@@ -208,6 +207,4 @@
       </inertial>
     </link>
-    <!-- Kobuki Gazebo simulation details -->
-    <!-- <kobuki_sim/> -->
   </xacro:macro>
 </robot>

File: robot_description/urdf/sensors/d435.urdf.xacro (robot description, xacro)
@@ -7,6 +7,6 @@
 -->
 <robot name="sensor_d435" xmlns:xacro="http://ros.org/wiki/xacro">
+  <xacro:include filename="$(find robot_description)/urdf/common_properties.urdf.xacro"/>
   <xacro:macro name="sensor_d435" params="parent *origin">
-    <xacro:property name="M_PI" value="3.1415926535897931" />
     <!-- The following values are approximate, and the camera node
      publishing TF values with actual calibrated camera extrinsic values -->
@@ -26,7 +26,4 @@
     <xacro:property name="d435_cam_depth_py" value="0.0175"/>
     <xacro:property name="d435_cam_depth_pz" value="${d435_cam_height/2}"/>
-    <material name="aluminum">
-	    <color rgba="0.5 0.5 0.5 1"/>
-    </material>
     <!-- camera body, with origin at bottom screw mount -->
     <joint name="camera_joint" type="fixed">
@@ -46,12 +43,12 @@
         <geometry>
           <!-- <box size="${d435_cam_width} ${d435_cam_height} ${d435_cam_depth}"/> -->
-          <mesh filename="package://robot_description/meshes/d435.dae" />
+          <mesh filename="package://robot_description/meshes/sensors/d435.dae" />
         </geometry>
-        <material name="aluminum"/>
+        <xacro:insert_block name="material_aluminum"/>
       </visual>
       <collision>
         <origin xyz="0 ${-d435_cam_depth_py} 0" rpy="0 0 0"/>
         <geometry>
-        <box size="${d435_cam_depth} ${d435_cam_width} ${d435_cam_height}"/>
+          <box size="${d435_cam_depth} ${d435_cam_width} ${d435_cam_height}"/>
         </geometry>
       </collision>
@@ -60,5 +57,7 @@
         <mass value="0.564" />
         <origin xyz="0 0 0" />
-        <inertia ixx="0.003881243" ixy="0.0" ixz="0.0" iyy="0.000498940" iyz="0.0" izz="0.003879257" />
+        <inertia ixx="0.003881243" ixy="0.0" ixz="0.0"
+                 iyy="0.000498940" iyz="0.0"
+                 izz="0.003879257" />
       </inertial>
     </link>

File: robot_description/urdf/sensors/rplidar.urdf.xacro (robot description, xacro)
@@ -1,36 +1,38 @@
 <?xml version="1.0"?>
-<robot xmlns:xacro="http://www.ros.org/wiki/xacro">
-    <xacro:macro name="rplidar_model" params="name parent *origin">
-      <joint name="${name}_joint" type="fixed">
-        <xacro:insert_block name="origin" />
-        <parent link="${parent}"/>
-        <child link="${name}_frame"/>
-      </joint>
-      <link name="${name}_frame">
-        <inertial>
-          <mass value="0.270" />
-          <origin xyz="0 0 0" rpy="0 0 0" />
-          <inertia ixx="2.632e-4" ixy="0" ixz="0"
-                   iyy="2.632e-4" iyz="0"
-                   izz="1.62e-4" />
-        </inertial>
-        <visual>
-          <origin xyz="0 0 0" rpy="0 0 0" />
-          <geometry>
-          <mesh filename="package://robot_description/meshes/rplidar_a2.stl"/>
+<robot xmlns:xacro="http://ros.org/wiki/xacro">
+  <xacro:include filename="$(find robot_description)/urdf/common_properties.urdf.xacro"/>
+  <xacro:macro name="rplidar_model" params="name parent *origin">
+    <joint name="${name}_joint" type="fixed">
+      <xacro:insert_block name="origin" />
+      <parent link="${parent}"/>
+      <child link="${name}_frame"/>
+    </joint>
+    <link name="${name}_frame">
+      <inertial>
+        <mass value="0.270" />
+        <origin xyz="0 0 0" rpy="0 0 0" />
+        <inertia ixx="2.632e-4" ixy="0" ixz="0"
+                 iyy="2.632e-4" iyz="0"
+                 izz="1.62e-4" />
+      </inertial>
+      <visual>
+        <origin xyz="0 0 0" rpy="0 0 1.5708" />
+        <geometry>
+          <mesh filename="package://robot_description/meshes/sensors/rplidar_a2.stl"/>
         </geometry>
-        </visual>
-        <collision>
-          <origin xyz="0 0 -0.0115" rpy="0 0 0" />
-          <geometry>
+        <xacro:insert_block name="material_dark_grey"/>
+      </visual>
+      <collision>
+        <origin xyz="0 0 -0.0115" rpy="0 0 0" />
+        <geometry>
           <box size="0.058 0.058 0.087" />
         </geometry>
-        </collision>
-      </link>
-    </xacro:macro>
-    <xacro:macro name="rplidar" params="name parent *origin ros_topic update_rate ray_count min_angle max_angle">
-      <xacro:rplidar_model name="${name}" parent="${parent}">
-        <xacro:insert_block name="origin" />
-      </xacro:rplidar_model>
-    </xacro:macro>
+      </collision>
+    </link>
+  </xacro:macro>
+  <xacro:macro name="rplidar" params="parent *origin">
+    <xacro:rplidar_model name="rplidar" parent="${parent}">
+      <xacro:insert_block name="origin" />
+    </xacro:rplidar_model>
+  </xacro:macro>
 </robot>

File: robot_description/urdf/stacks/custom_hexagons.urdf.xacro (robot description, xacro)
@@ -73,7 +73,9 @@
     <link name="pole_top_${number}_link">
       <visual>
-        <origin xyz=" 0 0 0" rpy="0 0 0"/>
+        <origin xyz="0 0 0" rpy="0 ${M_PI} 0"/>
         <geometry>
-          <mesh filename="package://robot_description/meshes/stacks/hexagons/pole_top.dae"/>
+          <!-- <mesh filename="package://robot_description/meshes/stacks/hexagons/pole_middle.dae"/> -->
+          <cylinder length="0.05" radius="0.003"/>
+          <xacro:insert_block name="material_aluminum"/>
         </geometry>
       </visual>
@@ -81,5 +83,5 @@
         <origin xyz="0 0 0" rpy="0 0 0"/>
         <geometry>
-          <cylinder length="0.2032" radius="0.006"/>
+          <cylinder length="0.05" radius="0.003"/>
         </geometry>
       </collision>
@@ -90,32 +92,4 @@
                  iyy="0.000206991" iyz="0.0"
                  izz="0.000001080"/>
-      </inertial>
-    </link>
-  </xacro:macro>
-  <xacro:macro name="stack_3d_sensor_pole" params="parent number x_loc y_loc z_loc">
-    <joint name="pole_kinect_${number}_joint" type="fixed">
-      <origin xyz="${x_loc} ${y_loc} ${z_loc}" rpy="0 0 0"/>
-      <parent link="${parent}"/>
-      <child link="pole_kinect_${number}_link"/>
-    </joint>
-    <link name="pole_kinect_${number}_link">
-      <visual>
-        <origin xyz="0 0 -0.01" rpy="0 0 0"/>
-        <geometry>
-          <mesh filename="package://robot_description/meshes/sensors/sensor_pole.dae" />
-        </geometry>
-      </visual>
-      <collision>
-        <origin xyz="0 0 0" rpy="0 0 0"/>
-        <geometry>
-          <cylinder length="0.0936" radius="0.006"/>
-        </geometry>
-      </collision>
-      <inertial>
-        <mass value="0.020"/>
-        <origin xyz="0 0 0"/>
-        <inertia ixx="0.000014782" ixy="0.0" ixz="0.0"
-                 iyy="0.000014782" iyz="0.0"
-                 izz="0.000000360"/>
       </inertial>
     </link>
@@ -172,5 +146,5 @@
         <origin xyz="0 0 0" rpy="0 0 0"/>
         <geometry>
-          <mesh filename="package://robot_description/meshes/stacks/hexagons/plate_middle.dae"/>
+          <mesh filename="package://robot_description/meshes/stacks/hexagons/plate_top.dae"/>
         </geometry>
       </visual>
@@ -189,12 +163,10 @@
       </inertial>
     </link>
-    <stack_top_pole parent="${parent}" number="0" x_loc= "0.0381" y_loc= "0.1505" z_loc="0.2920"/>
-    <stack_top_pole parent="${parent}" number="1" x_loc= "0.0381" y_loc="-0.1505" z_loc="0.2920"/>
-    <stack_top_pole parent="${parent}" number="2" x_loc="-0.0381" y_loc= "0.1505" z_loc="0.2920"/>
-    <stack_top_pole parent="${parent}" number="3" x_loc="-0.0381" y_loc="-0.1505" z_loc="0.2920"/>
-    <stack_3d_sensor_pole parent="${parent}" number="0" x_loc="-0.1024" y_loc= "0.098" z_loc="0.2372"/>
-    <stack_3d_sensor_pole parent="${parent}" number="1" x_loc="-0.1024" y_loc="-0.098" z_loc="0.2372"/>
+    <!-- <stack_top_pole parent="${parent}" number="0" x_loc= "0.0381" y_loc= "0.1505" z_loc="0.2252"/>
+    <stack_top_pole parent="${parent}" number="1" x_loc= "0.0381" y_loc="-0.1505" z_loc="0.2252"/>
+    <stack_top_pole parent="${parent}" number="2" x_loc="-0.0381" y_loc= "0.1505" z_loc="0.2252"/>
+    <stack_top_pole parent="${parent}" number="3" x_loc="-0.0381" y_loc="-0.1505" z_loc="0.2252"/>
     <joint name="plate_top_joint" type="fixed">
-      <origin xyz="-0.01364 0.0  0.3966" rpy="0 0 0"/>
+      <origin xyz="-0.01364 0.0 0" rpy="0 0 0"/>
       <parent link="${parent}"/>
       <child link="plate_top_link"/>
@@ -204,5 +176,5 @@
         <origin xyz="0 0 0" rpy="0 0 0"/>
         <geometry>
-          <mesh filename="package://robot_description/meshes/stacks/hexagons/plate_top.dae"/>
+          <mesh filename="package://robot_description/meshes/stacks/hexagons/plate_middle.dae"/>
         </geometry>
       </visual>
@@ -220,5 +192,5 @@
                  izz="0.006656" />
       </inertial>
-    </link>
+    </link> -->
   </xacro:macro>
 </robot>

Commit message: Next

File: robot_description/robots/kobuki_hexagons_d435.xacro (robot description, xacro)
@@ -18,5 +18,5 @@
   </sensor_d435>
   <rplidar parent="plate_middle_link">
-    <origin xyz="0 0 0.0025" rpy="0 0 0"/>
+    <origin xyz="0 0 0.0025" rpy="0 0 ${M_PI}"/>
   </rplidar>
 </robot>

File: robot_description/urdf/sensors/rplidar.urdf.xacro (robot description, xacro)
@@ -17,5 +17,5 @@
       </inertial>
       <visual>
-        <origin xyz="0 0 0" rpy="0 0 1.5708" />
+        <origin xyz="0 0 0" rpy="0 0 -${M_PI/2}" />
         <geometry>
           <mesh filename="package://robot_description/meshes/sensors/rplidar_a2.stl"/>
